File: canAIReGasSensorKit/canAIReSensor.brd (EAGLE design)
At the start: 54.6 x 35.6 mm, 23 parts, among them IC1 LP2951N, IC2 AD820N, Q1 FQN1N50CI, Q2 FQN1N50CI

Commit message: bundled for fab
Parts:
- added C5: (no value), rcl:C050-024X044
- added R7: 330k, rcl:0204/7
- added R8: 100, rcl:0204/7
- R1: value (none) -> 1.4k; device rcl:0207/10 -> rcl:0204/7
- R2: value (none) -> 357k; device rcl:0207/10 -> rcl:0204/7
- R3, R6: value (none) -> 10k; device rcl:0207/10 -> rcl:0204/7
- R4, R5: device rcl:0207/10 -> rcl:0204/7
- moved C2 2.84 mm to (23.5, 6.99)
- moved C4 2.84 mm to (21.0, 6.99)
- moved JP1 2.29 mm to (41.3, 8.26)
- moved C1 1.90 mm to (40.0, 13.3), turned to 90 degrees
- turned C3 to 180 degrees
Connections:
- new net N$7: IC1.5, R7.1
- new net N$9: IC2.2, IC2.6, R8.2
- net GND: now also C5.2
- net S2: now also IC2.3; no longer IC2.2
- net SENSOR: now also R8.1; no longer IC2.3, IC2.6
- net VCC: now also C5.1, R7.2
Routing:
- net N$9: track 0.00 -> 14.3 mm
- net SENSOR: track 21.6 -> 8.10 mm
- net VCC: track 45.2 -> 55.5 mm
- net S2: track 55.8 -> 52.9 mm
- net N$7: track 0.00 -> 2.54 mm
- net RANGE: track 32.2 -> 31.0 mm
- net HPWR: track 18.9 -> 19.6 mm
- net OVERHEAT: track 39.0 -> 39.6 mm
- net N$6: track 8.53 -> 8.00 mm
- net N$1: track 14.4 -> 15.0 mm
- net N$2: track 6.13 -> 6.66 mm
Other:
- outline, holes or cut-outs redrawn
