File: bGeigieNanoKit/bGeigieNanoKit.brd (EAGLE design)
At the start: 104.8 x 66.7 mm, 38 parts, among them T1 2SC1815

Commit message: final changes and output files for Rev. 2
Parts:
- removed JP6: (no value), SparkFun:SJ_2S-NO
- added SJ1: (no value), microbuilder:SOLDERJUMPER_CLOSEDWIRE
- moved R8 3.13 mm to (31.1, 23.8)
- moved R9 2.56 mm to (31.1, 26.4)
- moved JP2 0.71 mm to (19.1, 16.5)
- moved C3 0.45 mm to (47.0, 25.4)
- renumbered U$4 to S2
Connections:
- net VBATT: now also SJ1.2; no longer JP6.1
- net VGPS: now also SJ1.1; no longer JP6.2
Routing:
- net VBATT: track 96.5 -> 89.4 mm, vias 1 -> 3
- net N$24: track 15.4 -> 13.7 mm
- net VGPS: track 6.41 -> 7.37 mm
